File: hardware/BuReCon/busredundancycontroller/Power.sch (KiCad schematic (older format))
At the start: 23 parts, among them J1 USB_B_Micro, U1 ICE40LP1K-CM36, U2 AP7361C-33E, U3 AP7361C-12E

Commit message: House Keeping
House keeping
Parts:
- C1, C10, C11, C12, C2, C3, C4, C5, C6, C7, C8, C9: footprint (none) -> Capacitor_SMD:C_0201_0603Metric
- FB1: footprint (none) -> Fuse:Fuse_0603_1608Metric
- J1: footprint (none) -> Connector_USB:USB_Micro-AB_Molex_47590-0001
- LD1: footprint (none) -> LED_SMD:LED_0201_0603Metric
- R1: footprint (none) -> Resistor_SMD:R_0603_1608Metric
- TP1, TP2, TP3: footprint (none) -> TestPoint:TestPoint_Plated_Hole_D3.0mm
- U1: footprint UCBGA36_LAT -> ICE40LP1K-CM36:ICE40LP1K-CM36
Changed lines of the file:
@@
 F 0 "C2" H 3442 4196 50  0000 L CNN
 F 1 "100nF" H 3442 4105 50  0000 L CNN
-F 2 "" H 3350 4150 50  0001 C CNN
+F 2 "Capacitor_SMD:C_0201_0603Metric" H 3350 4150 50  0001 C CNN
 F 3 "~" H 3350 4150 50  0001 C CNN
 	1    3350 4150
@@
 F 0 "C3" H 3842 4196 50  0000 L CNN
 F 1 "100nF" H 3842 4105 50  0000 L CNN
-F 2 "" H 3750 4150 50  0001 C CNN
+F 2 "Capacitor_SMD:C_0201_0603Metric" H 3750 4150 50  0001 C CNN
 F 3 "~" H 3750 4150 50  0001 C CNN
 	1    3750 4150
@@
 F 0 "C4" H 4192 4196 50  0000 L CNN
 F 1 "100nF" H 4192 4105 50  0000 L CNN
-F 2 "" H 4100 4150 50  0001 C CNN
+F 2 "Capacitor_SMD:C_0201_0603Metric" H 4100 4150 50  0001 C CNN
 F 3 "~" H 4100 4150 50  0001 C CNN
 	1    4100 4150
@@
 F 0 "C5" H 4592 4196 50  0000 L CNN
 F 1 "100nF" H 4592 4105 50  0000 L CNN
-F 2 "" H 4500 4150 50  0001 C CNN
+F 2 "Capacitor_SMD:C_0201_0603Metric" H 4500 4150 50  0001 C CNN
 F 3 "~" H 4500 4150 50  0001 C CNN
 	1    4500 4150
@@
 F 0 "C6" H 5242 4196 50  0000 L CNN
 F 1 "100nF" H 5242 4105 50  0000 L CNN
-F 2 "" H 5150 4150 50  0001 C CNN
+F 2 "Capacitor_SMD:C_0201_0603Metric" H 5150 4150 50  0001 C CNN
 F 3 "~" H 5150 4150 50  0001 C CNN
 	1    5150 4150
@@
 F 0 "C7" H 5642 4196 50  0000 L CNN
 F 1 "100nF" H 5642 4105 50  0000 L CNN
-F 2 "" H 5550 4150 50  0001 C CNN
+F 2 "Capacitor_SMD:C_0201_0603Metric" H 5550 4150 50  0001 C CNN
 F 3 "~" H 5550 4150 50  0001 C CNN
 	1    5550 4150
@@
 F 0 "C8" H 6742 4196 50  0000 L CNN
 F 1 "100nF" H 6742 4105 50  0000 L CNN
-F 2 "" H 6650 4150 50  0001 C CNN
+F 2 "Capacitor_SMD:C_0201_0603Metric" H 6650 4150 50  0001 C CNN
 F 3 "~" H 6650 4150 50  0001 C CNN
 	1    6650 4150
@@
 F 0 "C9" H 7192 4196 50  0000 L CNN
 F 1 "100nF" H 7192 4105 50  0000 L CNN
-F 2 "" H 7100 4150 50  0001 C CNN
+F 2 "Capacitor_SMD:C_0201_0603Metric" H 7100 4150 50  0001 C CNN
 F 3 "~" H 7100 4150 50  0001 C CNN
 	1    7100 4150
@@
 F 0 "C10" H 8242 4196 50  0000 L CNN
 F 1 "100nF" H 8242 4105 50  0000 L CNN
-F 2 "" H 8150 4150 50  0001 C CNN
+F 2 "Capacitor_SMD:C_0201_0603Metric" H 8150 4150 50  0001 C CNN
 F 3 "~" H 8150 4150 50  0001 C CNN
 	1    8150 4150
@@
 F 0 "C11" H 3392 6596 50  0000 L CNN
 F 1 "4.7uF" H 3392 6505 50  0000 L CNN
-F 2 "" H 3300 6550 50  0001 C CNN
+F 2 "Capacitor_SMD:C_0201_0603Metric" H 3300 6550 50  0001 C CNN
 F 3 "~" H 3300 6550 50  0001 C CNN
 	1    3300 6550
@@
 F 0 "TP2" H 3560 6544 50  0000 L CNN
 F 1 "+3.3V" H 3560 6453 50  0000 L CNN
-F 2 "" H 3500 6450 50  0001 C CNN
+F 2 "TestPoint:TestPoint_Plated_Hole_D3.0mm" H 3500 6450 50  0001 C CNN
 F 3 "~" H 3500 6450 50  0001 C CNN
 	1    3300 6450
@@
 F 0 "C12" H 5592 6596 50  0000 L CNN
 F 1 "4.7uF" H 5592 6505 50  0000 L CNN
-F 2 "" H 5500 6550 50  0001 C CNN
+F 2 "Capacitor_SMD:C_0201_0603Metric" H 5500 6550 50  0001 C CNN
 F 3 "~" H 5500 6550 50  0001 C CNN
 	1    5500 6550
@@
 F 0 "TP1" V 10112 1140 50  0000 L CNN
 F 1 "5V" V 10203 1140 50  0000 L CNN
-F 2 "" H 10250 1000 50  0001 C CNN
+F 2 "TestPoint:TestPoint_Plated_Hole_D3.0mm" H 10250 1000 50  0001 C CNN
 F 3 "~" H 10250 1000 50  0001 C CNN
 	1    10050 1000
@@
 F 0 "J1" H 8007 2117 50  0000 C CNN
 F 1 "USB_B_Micro" H 8007 2026 50  0000 C CNN
-F 2 "" H 8100 1600 50  0001 C CNN
+F 2 "Connector_USB:USB_Micro-AB_Molex_47590-0001" H 8100 1600 50  0001 C CNN
 F 3 "~" H 8100 1600 50  0001 C CNN
 	1    7950 1650
@@
 F 0 "C1" H 8842 1146 50  0000 L CNN
 F 1 "100nF" H 8842 1055 50  0000 L CNN
-F 2 "" H 8750 1100 50  0001 C CNN
+F 2 "Capacitor_SMD:C_0201_0603Metric" H 8750 1100 50  0001 C CNN
 F 3 "~" H 8750 1100 50  0001 C CNN
 	1    8750 1100
@@
 F 0 "FB1" V 9263 1000 50  0000 C CNN
 F 1 "BLM18SG121TN1D" V 9354 1000 50  0000 C CNN
-F 2 "" V 9430 1000 50  0001 C CNN
+F 2 "Fuse:Fuse_0603_1608Metric" V 9430 1000 50  0001 C CNN
 F 3 "https://datasheet.octopart.com/BLM18SG121TN1D-Murata-datasheet-138707216.pdf" H 9500 1000 50  0001 C CNN
 	1    9500 1000
@@
 F 0 "TP3" H 5760 6544 50  0000 L CNN
 F 1 "1.2V" H 5760 6453 50  0000 L CNN
-F 2 "" H 5700 6450 50  0001 C CNN
+F 2 "TestPoint:TestPoint_Plated_Hole_D3.0mm" H 5700 6450 50  0001 C CNN
 F 3 "~" H 5700 6450 50  0001 C CNN
 	1    5500 6450
@@
 F 0 "R1" H 5859 1696 50  0000 L CNN
 F 1 "2k2 5% 0.063W" H 5859 1605 50  0000 L CNN
-F 2 "" H 5800 1650 50  0001 C CNN
+F 2 "Resistor_SMD:R_0603_1608Metric" H 5800 1650 50  0001 C CNN
 F 3 "~" H 5800 1650 50  0001 C CNN
 	1    5800 1650
@@
 F 0 "LD1" V 5839 1882 50  0000 R CNN
 F 1 "Blue" V 5748 1882 50  0000 R CNN
-F 2 "" H 5800 2000 50  0001 C CNN
+F 2 "LED_SMD:LED_0201_0603Metric" H 5800 2000 50  0001 C CNN
 F 3 "~" H 5800 2000 50  0001 C CNN
 	1    5800 2000
@@
 F 0 "U1" H 3500 1987 60  0000 C CNN
 F 1 "ICE40LP1K-CM36" H 3500 1881 60  0000 C CNN
-F 2 "UCBGA36_LAT" H 4000 1840 60  0001 C CNN
+F 2 "ICE40LP1K-CM36:ICE40LP1K-CM36" H 4000 1840 60  0001 C CNN
 F 3 "" H 2500 1500 60  0000 C CNN
 	2    2500 1500

Commit message: Connectors and RS232
Parts:
- LD1: value Blue -> Red
Changed lines of the file:
@@
 P 5800 2000
 F 0 "LD1" V 5839 1882 50  0000 R CNN
-F 1 "Blue" V 5748 1882 50  0000 R CNN
+F 1 "Red" V 5748 1882 50  0000 R CNN
 F 2 "LED_SMD:LED_0201_0603Metric" H 5800 2000 50  0001 C CNN
 F 3 "~" H 5800 2000 50  0001 C CNN

Commit message: Footprints, Initial PCB
Parts:
- C1, C10, C11, C12, C2, C3, C4, C5, C6, C7, C8, C9: footprint Capacitor_SMD:C_0201_0603Metric -> Capacitor_SMD:C_0603_1608Metric
- FB1: footprint Fuse:Fuse_0603_1608Metric -> Inductor_SMD:L_0603_1608Metric
- LD1: footprint LED_SMD:LED_0201_0603Metric -> LED_SMD:LED_0603_1608Metric
- TP1, TP2, TP3: footprint TestPoint:TestPoint_Plated_Hole_D3.0mm -> TestPoint:TestPoint_Pad_D1.0mm
- U2, U3: footprint Package_TO_SOT_SMD:SOT-223-3_TabPin2 -> Package_TO_SOT_SMD:SOT-223
Changed lines of the file:
@@
 F 0 "C2" H 3442 4196 50  0000 L CNN
 F 1 "100nF" H 3442 4105 50  0000 L CNN
-F 2 "Capacitor_SMD:C_0201_0603Metric" H 3350 4150 50  0001 C CNN
+F 2 "Capacitor_SMD:C_0603_1608Metric" H 3350 4150 50  0001 C CNN
 F 3 "~" H 3350 4150 50  0001 C CNN
 	1    3350 4150
@@
 F 0 "C3" H 3842 4196 50  0000 L CNN
 F 1 "100nF" H 3842 4105 50  0000 L CNN
-F 2 "Capacitor_SMD:C_0201_0603Metric" H 3750 4150 50  0001 C CNN
+F 2 "Capacitor_SMD:C_0603_1608Metric" H 3750 4150 50  0001 C CNN
 F 3 "~" H 3750 4150 50  0001 C CNN
 	1    3750 4150
@@
 F 0 "C4" H 4192 4196 50  0000 L CNN
 F 1 "100nF" H 4192 4105 50  0000 L CNN
-F 2 "Capacitor_SMD:C_0201_0603Metric" H 4100 4150 50  0001 C CNN
+F 2 "Capacitor_SMD:C_0603_1608Metric" H 4100 4150 50  0001 C CNN
 F 3 "~" H 4100 4150 50  0001 C CNN
 	1    4100 4150
@@
 F 0 "C5" H 4592 4196 50  0000 L CNN
 F 1 "100nF" H 4592 4105 50  0000 L CNN
-F 2 "Capacitor_SMD:C_0201_0603Metric" H 4500 4150 50  0001 C CNN
+F 2 "Capacitor_SMD:C_0603_1608Metric" H 4500 4150 50  0001 C CNN
 F 3 "~" H 4500 4150 50  0001 C CNN
 	1    4500 4150
@@
 F 0 "C6" H 5242 4196 50  0000 L CNN
 F 1 "100nF" H 5242 4105 50  0000 L CNN
-F 2 "Capacitor_SMD:C_0201_0603Metric" H 5150 4150 50  0001 C CNN
+F 2 "Capacitor_SMD:C_0603_1608Metric" H 5150 4150 50  0001 C CNN
 F 3 "~" H 5150 4150 50  0001 C CNN
 	1    5150 4150
@@
 F 0 "C7" H 5642 4196 50  0000 L CNN
 F 1 "100nF" H 5642 4105 50  0000 L CNN
-F 2 "Capacitor_SMD:C_0201_0603Metric" H 5550 4150 50  0001 C CNN
+F 2 "Capacitor_SMD:C_0603_1608Metric" H 5550 4150 50  0001 C CNN
 F 3 "~" H 5550 4150 50  0001 C CNN
 	1    5550 4150
@@
 F 0 "C8" H 6742 4196 50  0000 L CNN
 F 1 "100nF" H 6742 4105 50  0000 L CNN
-F 2 "Capacitor_SMD:C_0201_0603Metric" H 6650 4150 50  0001 C CNN
+F 2 "Capacitor_SMD:C_0603_1608Metric" H 6650 4150 50  0001 C CNN
 F 3 "~" H 6650 4150 50  0001 C CNN
 	1    6650 4150
@@
 F 0 "C9" H 7192 4196 50  0000 L CNN
 F 1 "100nF" H 7192 4105 50  0000 L CNN
-F 2 "Capacitor_SMD:C_0201_0603Metric" H 7100 4150 50  0001 C CNN
+F 2 "Capacitor_SMD:C_0603_1608Metric" H 7100 4150 50  0001 C CNN
 F 3 "~" H 7100 4150 50  0001 C CNN
 	1    7100 4150
@@
 F 0 "C10" H 8242 4196 50  0000 L CNN
 F 1 "100nF" H 8242 4105 50  0000 L CNN
-F 2 "Capacitor_SMD:C_0201_0603Metric" H 8150 4150 50  0001 C CNN
+F 2 "Capacitor_SMD:C_0603_1608Metric" H 8150 4150 50  0001 C CNN
 F 3 "~" H 8150 4150 50  0001 C CNN
 	1    8150 4150
@@
 F 0 "U2" H 2700 6692 50  0000 C CNN
 F 1 "AP7361C-33E" H 2700 6601 50  0000 C CNN
-F 2 "Package_TO_SOT_SMD:SOT-223-3_TabPin2" H 2700 6675 50  0001 C CIN
+F 2 "Package_TO_SOT_SMD:SOT-223" H 2700 6675 50  0001 C CIN
 F 3 "https://www.diodes.com/assets/Datasheets/AP7361C.pdf" H 2700 6400 50  0001 C CNN
 	1    2700 6450
@@
 F 0 "C11" H 3392 6596 50  0000 L CNN
 F 1 "4.7uF" H 3392 6505 50  0000 L CNN
-F 2 "Capacitor_SMD:C_0201_0603Metric" H 3300 6550 50  0001 C CNN
+F 2 "Capacitor_SMD:C_0603_1608Metric" H 3300 6550 50  0001 C CNN
 F 3 "~" H 3300 6550 50  0001 C CNN
 	1    3300 6550
@@
 F 0 "TP2" H 3560 6544 50  0000 L CNN
 F 1 "+3.3V" H 3560 6453 50  0000 L CNN
-F 2 "TestPoint:TestPoint_Plated_Hole_D3.0mm" H 3500 6450 50  0001 C CNN
+F 2 "TestPoint:TestPoint_Pad_D1.0mm" H 3500 6450 50  0001 C CNN
 F 3 "~" H 3500 6450 50  0001 C CNN
 	1    3300 6450
@@
 F 0 "U3" H 4900 6692 50  0000 C CNN
 F 1 "AP7361C-12E" H 4900 6601 50  0000 C CNN
-F 2 "Package_TO_SOT_SMD:SOT-223-3_TabPin2" H 4900 6675 50  0001 C CIN
+F 2 "Package_TO_SOT_SMD:SOT-223" H 4900 6675 50  0001 C CIN
 F 3 "https://www.diodes.com/assets/Datasheets/AP7361C.pdf" H 4900 6400 50  0001 C CNN
 	1    4900 6450
@@
 F 0 "C12" H 5592 6596 50  0000 L CNN
 F 1 "4.7uF" H 5592 6505 50  0000 L CNN
-F 2 "Capacitor_SMD:C_0201_0603Metric" H 5500 6550 50  0001 C CNN
+F 2 "Capacitor_SMD:C_0603_1608Metric" H 5500 6550 50  0001 C CNN
 F 3 "~" H 5500 6550 50  0001 C CNN
 	1    5500 6550
@@
 F 0 "TP1" V 10112 1140 50  0000 L CNN
 F 1 "5V" V 10203 1140 50  0000 L CNN
-F 2 "TestPoint:TestPoint_Plated_Hole_D3.0mm" H 10250 1000 50  0001 C CNN
+F 2 "TestPoint:TestPoint_Pad_D1.0mm" H 10250 1000 50  0001 C CNN
 F 3 "~" H 10250 1000 50  0001 C CNN
 	1    10050 1000
@@
 F 0 "C1" H 8842 1146 50  0000 L CNN
 F 1 "100nF" H 8842 1055 50  0000 L CNN
-F 2 "Capacitor_SMD:C_0201_0603Metric" H 8750 1100 50  0001 C CNN
+F 2 "Capacitor_SMD:C_0603_1608Metric" H 8750 1100 50  0001 C CNN
 F 3 "~" H 8750 1100 50  0001 C CNN
 	1    8750 1100
@@
 F 0 "FB1" V 9263 1000 50  0000 C CNN
 F 1 "BLM18SG121TN1D" V 9354 1000 50  0000 C CNN
-F 2 "Fuse:Fuse_0603_1608Metric" V 9430 1000 50  0001 C CNN
+F 2 "Inductor_SMD:L_0603_1608Metric" V 9430 1000 50  0001 C CNN
 F 3 "https://datasheet.octopart.com/BLM18SG121TN1D-Murata-datasheet-138707216.pdf" H 9500 1000 50  0001 C CNN
 	1    9500 1000
@@
 F 0 "TP3" H 5760 6544 50  0000 L CNN
 F 1 "1.2V" H 5760 6453 50  0000 L CNN
-F 2 "TestPoint:TestPoint_Plated_Hole_D3.0mm" H 5700 6450 50  0001 C CNN
+F 2 "TestPoint:TestPoint_Pad_D1.0mm" H 5700 6450 50  0001 C CNN
 F 3 "~" H 5700 6450 50  0001 C CNN
 	1    5500 6450
@@
 F 0 "LD1" V 5839 1882 50  0000 R CNN
 F 1 "Red" V 5748 1882 50  0000 R CNN
-F 2 "LED_SMD:LED_0201_0603Metric" H 5800 2000 50  0001 C CNN
+F 2 "LED_SMD:LED_0603_1608Metric" H 5800 2000 50  0001 C CNN
 F 3 "~" H 5800 2000 50  0001 C CNN
 	1    5800 2000
