File: hardware/BuReCon/busredundancycontroller/USB_SERIAL.sch (KiCad schematic (older format))
At the start: 31 parts, among them U4 USBLC6-2SC6, U5 FT2232HL, U6 93LC56C, U7 DSC1001DI1

Commit message: Footprints, Initial PCB
Parts:
- C13, C14, C15, C16, C17, C18, C19, C20, C21, C22, C23, C24, C25, C26, C27: footprint Capacitor_SMD:C_0201_0603Metric -> Capacitor_SMD:C_0603_1608Metric
- FB2, FB3: footprint Fuse:Fuse_0603_1608Metric -> Inductor_SMD:L_0603_1608Metric
- LD3, LD4: footprint LED_SMD:LED_0201_0603Metric -> LED_SMD:LED_0603_1608Metric
- U6: footprint Package_TO_SOT_SMD:SOT-23-8 -> Package_SO:SOIC-8_3.9x4.9mm_P1.27mm
Changed lines of the file:
@@
 F 0 "C21" H 9042 1846 50  0000 L CNN
 F 1 "100nF" H 9042 1755 50  0000 L CNN
-F 2 "Capacitor_SMD:C_0201_0603Metric" H 8950 1800 50  0001 C CNN
+F 2 "Capacitor_SMD:C_0603_1608Metric" H 8950 1800 50  0001 C CNN
 F 3 "~" H 8950 1800 50  0001 C CNN
 	1    8950 1800
@@
 F 0 "C22" H 9442 1846 50  0000 L CNN
 F 1 "100nF" H 9442 1755 50  0000 L CNN
-F 2 "Capacitor_SMD:C_0201_0603Metric" H 9350 1800 50  0001 C CNN
+F 2 "Capacitor_SMD:C_0603_1608Metric" H 9350 1800 50  0001 C CNN
 F 3 "~" H 9350 1800 50  0001 C CNN
 	1    9350 1800
@@
 F 0 "C23" H 9842 1846 50  0000 L CNN
 F 1 "100nF" H 9842 1755 50  0000 L CNN
-F 2 "Capacitor_SMD:C_0201_0603Metric" H 9750 1800 50  0001 C CNN
+F 2 "Capacitor_SMD:C_0603_1608Metric" H 9750 1800 50  0001 C CNN
 F 3 "~" H 9750 1800 50  0001 C CNN
 	1    9750 1800
@@
 F 0 "C20" H 8642 1846 50  0000 L CNN
 F 1 "100nF" H 8642 1755 50  0000 L CNN
-F 2 "Capacitor_SMD:C_0201_0603Metric" H 8550 1800 50  0001 C CNN
+F 2 "Capacitor_SMD:C_0603_1608Metric" H 8550 1800 50  0001 C CNN
 F 3 "~" H 8550 1800 50  0001 C CNN
 	1    8550 1800
@@
 F 0 "FB2" V 4400 950 50  0000 C CNN
 F 1 "BLM18SG121TN1D" V 4700 900 50  0000 C CNN
-F 2 "Fuse:Fuse_0603_1608Metric" V 4480 950 50  0001 C CNN
+F 2 "Inductor_SMD:L_0603_1608Metric" V 4480 950 50  0001 C CNN
 F 3 "https://datasheet.octopart.com/BLM18SG121TN1D-Murata-datasheet-138707216.pdf" H 4550 950 50  0001 C CNN
 	1    4550 950
@@
 F 0 "FB3" V 3900 1650 50  0000 C CNN
 F 1 "BLM18SG121TN1D" V 4200 1450 50  0000 C CNN
-F 2 "Fuse:Fuse_0603_1608Metric" V 3980 1650 50  0001 C CNN
+F 2 "Inductor_SMD:L_0603_1608Metric" V 3980 1650 50  0001 C CNN
 F 3 "https://datasheet.octopart.com/BLM18SG121TN1D-Murata-datasheet-138707216.pdf" H 4050 1650 50  0001 C CNN
 	1    4050 1650
@@
 F 0 "C16" H 5092 1146 50  0000 L CNN
 F 1 "10nF" H 5092 1055 50  0000 L CNN
-F 2 "Capacitor_SMD:C_0201_0603Metric" H 5000 1100 50  0001 C CNN
+F 2 "Capacitor_SMD:C_0603_1608Metric" H 5000 1100 50  0001 C CNN
 F 3 "~" H 5000 1100 50  0001 C CNN
 	1    5000 1100
@@
 F 0 "C17" H 5492 1146 50  0000 L CNN
 F 1 "100nF" H 5492 1055 50  0000 L CNN
-F 2 "Capacitor_SMD:C_0201_0603Metric" H 5400 1100 50  0001 C CNN
+F 2 "Capacitor_SMD:C_0603_1608Metric" H 5400 1100 50  0001 C CNN
 F 3 "~" H 5400 1100 50  0001 C CNN
 	1    5400 1100
@@
 F 0 "C18" H 4392 1796 50  0000 L CNN
 F 1 "10nF" H 4392 1705 50  0000 L CNN
-F 2 "Capacitor_SMD:C_0201_0603Metric" H 4300 1750 50  0001 C CNN
+F 2 "Capacitor_SMD:C_0603_1608Metric" H 4300 1750 50  0001 C CNN
 F 3 "~" H 4300 1750 50  0001 C CNN
 	1    4300 1750
@@
 F 0 "C19" H 4842 1796 50  0000 L CNN
 F 1 "100nF" H 4842 1705 50  0000 L CNN
-F 2 "Capacitor_SMD:C_0201_0603Metric" H 4750 1750 50  0001 C CNN
+F 2 "Capacitor_SMD:C_0603_1608Metric" H 4750 1750 50  0001 C CNN
 F 3 "~" H 4750 1750 50  0001 C CNN
 	1    4750 1750
@@
 F 0 "C24" H 3592 2346 50  0000 L CNN
 F 1 "100nF" H 3592 2255 50  0000 L CNN
-F 2 "Capacitor_SMD:C_0201_0603Metric" H 3500 2300 50  0001 C CNN
+F 2 "Capacitor_SMD:C_0603_1608Metric" H 3500 2300 50  0001 C CNN
 F 3 "~" H 3500 2300 50  0001 C CNN
 	1    3500 2300
@@
 F 0 "C27" V 1550 6250 50  0000 L CNN
 F 1 "100nF" V 1750 6150 50  0000 L CNN
-F 2 "Capacitor_SMD:C_0201_0603Metric" H 1650 6350 50  0001 C CNN
+F 2 "Capacitor_SMD:C_0603_1608Metric" H 1650 6350 50  0001 C CNN
 F 3 "~" H 1650 6350 50  0001 C CNN
 	1    1650 6350
@@
 F 0 "U6" H 2050 4950 50  0000 C CNN
 F 1 "93LC56C" H 2200 4450 50  0000 C CNN
-F 2 "Package_TO_SOT_SMD:SOT-23-8" H 1950 4700 50  0001 C CNN
+F 2 "Package_SO:SOIC-8_3.9x4.9mm_P1.27mm" H 1950 4700 50  0001 C CNN
 F 3 "http://ww1.microchip.com/downloads/en/DeviceDoc/20001749K.pdf" H 1950 4700 50  0001 C CNN
 	1    1950 4700
@@
 F 0 "C26" H 1242 5046 50  0000 L CNN
 F 1 "100nF" H 1242 4955 50  0000 L CNN
-F 2 "Capacitor_SMD:C_0201_0603Metric" H 1150 5000 50  0001 C CNN
+F 2 "Capacitor_SMD:C_0603_1608Metric" H 1150 5000 50  0001 C CNN
 F 3 "~" H 1150 5000 50  0001 C CNN
 	1    1150 5000
@@
 F 0 "C13" H 6392 996 50  0000 L CNN
 F 1 "100nF" H 6392 905 50  0000 L CNN
-F 2 "Capacitor_SMD:C_0201_0603Metric" H 6300 950 50  0001 C CNN
+F 2 "Capacitor_SMD:C_0603_1608Metric" H 6300 950 50  0001 C CNN
 F 3 "~" H 6300 950 50  0001 C CNN
 	1    6300 950
@@
 F 0 "C14" H 6792 996 50  0000 L CNN
 F 1 "100nF" H 6792 905 50  0000 L CNN
-F 2 "Capacitor_SMD:C_0201_0603Metric" H 6700 950 50  0001 C CNN
+F 2 "Capacitor_SMD:C_0603_1608Metric" H 6700 950 50  0001 C CNN
 F 3 "~" H 6700 950 50  0001 C CNN
 	1    6700 950
@@
 F 0 "C15" H 7192 996 50  0000 L CNN
 F 1 "100nF" H 7192 905 50  0000 L CNN
-F 2 "Capacitor_SMD:C_0201_0603Metric" H 7100 950 50  0001 C CNN
+F 2 "Capacitor_SMD:C_0603_1608Metric" H 7100 950 50  0001 C CNN
 F 3 "~" H 7100 950 50  0001 C CNN
 	1    7100 950
@@
 F 0 "C25" H 4442 2646 50  0000 L CNN
 F 1 "10nF" H 4442 2555 50  0000 L CNN
-F 2 "Capacitor_SMD:C_0201_0603Metric" H 4350 2600 50  0001 C CNN
+F 2 "Capacitor_SMD:C_0603_1608Metric" H 4350 2600 50  0001 C CNN
 F 3 "~" H 4350 2600 50  0001 C CNN
 	1    4350 2600
@@
 F 0 "LD3" H 8850 5250 50  0000 R CNN
 F 1 "Yellow" H 8850 5050 50  0000 R CNN
-F 2 "LED_SMD:LED_0201_0603Metric" H 8700 5150 50  0001 C CNN
+F 2 "LED_SMD:LED_0603_1608Metric" H 8700 5150 50  0001 C CNN
 F 3 "~" H 8700 5150 50  0001 C CNN
 	1    8700 5150
@@
 F 0 "LD4" H 9650 5550 50  0000 R CNN
 F 1 "Green" H 9650 5350 50  0000 R CNN
-F 2 "LED_SMD:LED_0201_0603Metric" H 9500 5450 50  0001 C CNN
+F 2 "LED_SMD:LED_0603_1608Metric" H 9500 5450 50  0001 C CNN
 F 3 "~" H 9500 5450 50  0001 C CNN
 	1    9500 5450
