File: hardware/BuReCon/busredundancycontroller/connectors.sch (KiCad schematic (older format))
At the start: 15 parts, among them J2 Clock Output, J3 Differential IO, J4 Input/Output 1, J5 Input/Output 2, J6 Input/Output 3, J7 Input/Output 4, J8 Input/Output 5

Commit message: Footprints, Initial PCB
Parts:
- FID1, FID2, FID3, FID4: footprint (none) -> Fiducial:Fiducial_0.5mm_Mask1.5mm
- J2: footprint (none) -> Connector_PinHeader_1.00mm:PinHeader_1x01_P1.00mm_Vertical
- J3: footprint (none) -> Connector_PinHeader_1.00mm:PinHeader_1x06_P1.00mm_Vertical
- J4, J5, J6, J7, J8: footprint (none) -> Connector_PinHeader_1.00mm:PinHeader_1x02_P1.00mm_Vertical
- JP1, JP2: footprint (none) -> Jumper:SolderJumper-2_P1.3mm_Open_Pad1.0x1.5mm
- R20, R21: footprint (none) -> Resistor_SMD:R_0603_1608Metric
Changed lines of the file:
@@
 F 0 "JP1" H 3400 5014 50  0000 C CNN
 F 1 "CBSEL0" H 3400 4923 50  0000 C CNN
-F 2 "" H 3400 4750 50  0001 C CNN
+F 2 "Jumper:SolderJumper-2_P1.3mm_Open_Pad1.0x1.5mm" H 3400 4750 50  0001 C CNN
 F 3 "~" H 3400 4750 50  0001 C CNN
 	1    3400 4750
@@
 F 0 "JP2" H 3400 5564 50  0000 C CNN
 F 1 "CBSEL1" H 3400 5473 50  0000 C CNN
-F 2 "" H 3400 5300 50  0001 C CNN
+F 2 "Jumper:SolderJumper-2_P1.3mm_Open_Pad1.0x1.5mm" H 3400 5300 50  0001 C CNN
 F 3 "~" H 3400 5300 50  0001 C CNN
 	1    3400 5300
@@
 F 0 "R21" H 2859 4496 50  0000 L CNN
 F 1 "10k" H 2859 4405 50  0000 L CNN
-F 2 "" H 2800 4450 50  0001 C CNN
+F 2 "Resistor_SMD:R_0603_1608Metric" H 2800 4450 50  0001 C CNN
 F 3 "~" H 2800 4450 50  0001 C CNN
 	1    2800 4450
@@
 F 0 "R20" H 2459 4496 50  0000 L CNN
 F 1 "10k" H 2459 4405 50  0000 L CNN
-F 2 "" H 2400 4450 50  0001 C CNN
+F 2 "Resistor_SMD:R_0603_1608Metric" H 2400 4450 50  0001 C CNN
 F 3 "~" H 2400 4450 50  0001 C CNN
 	1    2400 4450
@@
 F 0 "J3" H 2318 1775 50  0000 C CNN
 F 1 "Differential IO" H 2318 1866 50  0000 C CNN
-F 2 "" H 2400 2300 50  0001 C CNN
+F 2 "Connector_PinHeader_1.00mm:PinHeader_1x06_P1.00mm_Vertical" H 2400 2300 50  0001 C CNN
 F 3 "~" H 2400 2300 50  0001 C CNN
 	1    2400 2300
@@
 F 0 "J6" H 7450 3350 50  0000 C CNN
 F 1 "Input/Output 3" H 7550 3650 50  0000 C CNN
-F 2 "" H 7500 3550 50  0001 C CNN
+F 2 "Connector_PinHeader_1.00mm:PinHeader_1x02_P1.00mm_Vertical" H 7500 3550 50  0001 C CNN
 F 3 "~" H 7500 3550 50  0001 C CNN
 	1    7500 3550
@@
 F 0 "J7" H 7450 4000 50  0000 C CNN
 F 1 "Input/Output 4" H 7550 4300 50  0000 C CNN
-F 2 "" H 7500 4200 50  0001 C CNN
+F 2 "Connector_PinHeader_1.00mm:PinHeader_1x02_P1.00mm_Vertical" H 7500 4200 50  0001 C CNN
 F 3 "~" H 7500 4200 50  0001 C CNN
 	1    7500 4200
@@
 F 0 "J5" H 7450 2750 50  0000 C CNN
 F 1 "Input/Output 2" H 7500 3050 50  0000 C CNN
-F 2 "" H 7500 2950 50  0001 C CNN
+F 2 "Connector_PinHeader_1.00mm:PinHeader_1x02_P1.00mm_Vertical" H 7500 2950 50  0001 C CNN
 F 3 "~" H 7500 2950 50  0001 C CNN
 	1    7500 2950
@@
 F 0 "J8" H 7450 4650 50  0000 C CNN
 F 1 "Input/Output 5" H 7550 4950 50  0000 C CNN
-F 2 "" H 7500 4850 50  0001 C CNN
+F 2 "Connector_PinHeader_1.00mm:PinHeader_1x02_P1.00mm_Vertical" H 7500 4850 50  0001 C CNN
 F 3 "~" H 7500 4850 50  0001 C CNN
 	1    7500 4850
@@
 F 0 "J4" H 7450 2150 50  0000 C CNN
 F 1 "Input/Output 1" H 7500 2450 50  0000 C CNN
-F 2 "" H 7500 2350 50  0001 C CNN
+F 2 "Connector_PinHeader_1.00mm:PinHeader_1x02_P1.00mm_Vertical" H 7500 2350 50  0001 C CNN
 F 3 "~" H 7500 2350 50  0001 C CNN
 	1    7500 2350
@@
 F 0 "J2" H 7450 1650 50  0000 C CNN
 F 1 "Clock Output" H 7500 1850 50  0000 C CNN
-F 2 "" H 7500 1750 50  0001 C CNN
+F 2 "Connector_PinHeader_1.00mm:PinHeader_1x01_P1.00mm_Vertical" H 7500 1750 50  0001 C CNN
 F 3 "~" H 7500 1750 50  0001 C CNN
 	1    7500 1750
@@
 F 0 "FID1" H 5235 6746 50  0000 L CNN
 F 1 "Fiducial" H 5235 6655 50  0000 L CNN
-F 2 "" H 5150 6700 50  0001 C CNN
+F 2 "Fiducial:Fiducial_0.5mm_Mask1.5mm" H 5150 6700 50  0001 C CNN
 F 3 "~" H 5150 6700 50  0001 C CNN
 	1    5150 6700
@@
 F 0 "FID2" H 5835 6746 50  0000 L CNN
 F 1 "Fiducial" H 5835 6655 50  0000 L CNN
-F 2 "" H 5750 6700 50  0001 C CNN
+F 2 "Fiducial:Fiducial_0.5mm_Mask1.5mm" H 5750 6700 50  0001 C CNN
 F 3 "~" H 5750 6700 50  0001 C CNN
 	1    5750 6700
@@
 F 0 "FID3" H 5235 7096 50  0000 L CNN
 F 1 "Fiducial" H 5235 7005 50  0000 L CNN
-F 2 "" H 5150 7050 50  0001 C CNN
+F 2 "Fiducial:Fiducial_0.5mm_Mask1.5mm" H 5150 7050 50  0001 C CNN
 F 3 "~" H 5150 7050 50  0001 C CNN
 	1    5150 7050
@@
 F 0 "FID4" H 5835 7096 50  0000 L CNN
 F 1 "Fiducial" H 5835 7005 50  0000 L CNN
-F 2 "" H 5750 7050 50  0001 C CNN
+F 2 "Fiducial:Fiducial_0.5mm_Mask1.5mm" H 5750 7050 50  0001 C CNN
 F 3 "~" H 5750 7050 50  0001 C CNN
 	1    5750 7050
